File: CARLOS.kicad_sch (KiCad schematic)
At the start: 1 part, among them U1 Heltec_ESP32_LoRa_V3

Commit message: Esquematico general del proyecto
Parts:
- added J1: PH, Connector_PinSocket_2.54mm:PinSocket_1x03_P2.54mm_Vertical, symbol Connector:Conn_01x03_Socket
- added J2: Conductividad, Connector_PinHeader_2.54mm:PinHeader_1x03_P2.54mm_Vertical, symbol Connector:Conn_01x03_Pin
- added J3: Humedad, Connector_PinSocket_1.00mm:PinSocket_1x04_P1.00mm_Vertical, symbol Connector:Conn_01x04_Socket
- added J4: BME280, TerminalBlock:TerminalBlock_MaiXu_MX126-5.0-04P_1x04_P5.00mm, symbol Connector:Screw_Terminal_01x04
- added J5: BH1750, Connector_PinHeader_2.54mm:PinHeader_1x05_P2.54mm_Vertical, symbol Connector:Conn_01x05_Socket
Connections:
- net GND: now reaches U1.J2_1 (GND_J2)
- net GND: now also J1.3 (Pin_3), J2.3 (Pin_3), J3.2 (Pin_2), J4.2 (Pin_2), J5.2 (Pin_2)
- net GPIO4: now reaches U1.J2_15 (GPIO4/ADC1_CH3/TOUCH4)
- net GPIO4: now also J1.2 (Pin_2)
- net GPIO3: now reaches U1.J2_16 (GPIO3/ADC1_CH2/TOUCH3)
- net GPIO3: now also J2.2 (Pin_2)
- net GPIO2: now reaches U1.J2_17 (GPIO2/ADC1_CH1/TOUCH2)
- net GPIO2: now also J3.4 (Pin_4)
- net +5V: now reaches U1.J2_2 (5V)
- net GPIO41: now reaches U1.J3_15 (GPIO41/MTDI)
- net GPIO41: now also J4.3 (Pin_3), J5.4 (Pin_4)
- net GPIO42: now reaches U1.J3_16 (GPIO42/MTMS)
- net GPIO42: now also J4.4 (Pin_4), J5.3 (Pin_3)
- new net +3.3V: J1.1 (Pin_1), J2.1 (Pin_1), J3.1 (Pin_1), J4.1 (Pin_1), J5.1 (Pin_1)
- no-connect marks 0 -> 2

Commit message: hola
Parts:
- added J6: Max485 to Micro, Connector_PinSocket_2.54mm:PinSocket_1x04_P2.54mm_Vertical, symbol Connector:Conn_01x04_Socket
- added J7: VCC to Max485, Connector_PinSocket_2.54mm:PinSocket_1x04_P2.54mm_Vertical, symbol Connector:Conn_01x04_Socket
Connections:
- net 3V3 is gone; now on net +3.3V: U1.J3_2 (3V3), U1.J3_3 (3V3)
- net +3.3V: now also J7.1 (Pin_1)
- net GND: now also U1.J3_1 (GND_J3), J7.4 (Pin_4)
- net GPIO7: now reaches U1.J2_12 (GPIO7/ADC1_CH6/TOUCH7)
- net GPIO7: now also J6.4 (Pin_4)
- net GPIO6: now reaches U1.J2_13 (GPIO6/ADC1_CH5/TOUCH6)
- net GPIO6: now also J6.1 (Pin_1)
- net GPIO5: now reaches U1.J2_14 (GPIO5/ADC1_CH4/TOUCH5)
- net GPIO5: now also J6.2 (Pin_2), J6.3 (Pin_3)

Commit message: PCB Finalizado
Parts:
- removed U1: Heltec_ESP32_LoRa_V3, Heltec_ESP32_LoRa_V3:Heltec_ESP32_LoRa_V3, symbol Heltec_ESP32_LoRa_V3:Heltec_ESP32_LoRa_V3
- added J2: DER, Connector_PinSocket_2.54mm:PinSocket_1x18_P2.54mm_Vertical, symbol Connector:Conn_01x18_Socket
- added J3: IZQ, Connector_PinSocket_2.54mm:PinSocket_1x18_P2.54mm_Vertical, symbol Connector:Conn_01x18_Socket
- added J8: NPK, TerminalBlock_MetzConnect:TerminalBlock_MetzConnect_Type055_RT01503HDWU_1x03_P5.00mm_Horizontal, symbol Connector:Screw_Terminal_01x03
- J4: footprint TerminalBlock:TerminalBlock_MaiXu_MX126-5.0-04P_1x04_P5.00mm -> TerminalBlock_MetzConnect:TerminalBlock_MetzConnect_Type055_RT01504HDWU_1x04_P5.00mm_Horizontal
- J9: renamed from J3; footprint Connector_PinSocket_1.00mm:PinSocket_1x04_P1.00mm_Vertical -> Connector_PinSocket_2.54mm:PinSocket_1x04_P2.54mm_Vertical
- renumbered J2 to J10
Connections:
- net +3.3V: now also J3.2 (Pin_2), J3.3 (Pin_3)
- net +5V: now also J2.2 (Pin_2)
- net GND: now also J2.1 (Pin_1), J3.1 (Pin_1), J8.1 (Pin_1)
- net GPIO2: now also J3.13 (Pin_13)
- net GPIO3: now also J3.14 (Pin_14)
- net GPIO4: now also J3.15 (Pin_15)
- net GPIO41: now also J3.8 (Pin_8)
- net GPIO42: now also J3.7 (Pin_7)
- net GPIO5: now also J3.16 (Pin_16)
- net GPIO6: now also J3.17 (Pin_17)
- net GPIO7: now also J3.18 (Pin_18)
- net B: now reaches J7.2 (Pin_2)
- net B: now also J8.3 (Pin_3)
- net A: now reaches J7.3 (Pin_3)
- net A: now also J8.2 (Pin_2)
Other:
- moved on the sheet: J6, J7
